Commit message: update in drone

File: src/drone/urdf/robot.urdf (robot description, URDF)
Before this commit: robot simple_box, 3 links, 2 joints
Links:
- added link arm_bl; visual cylinder length=0.3 radius=0.01
- added link arm_br; visual cylinder length=0.3 radius=0.01
- added link arm_fl; visual cylinder length=0.3 radius=0.01
- added link arm_fr; visual cylinder length=0.3 radius=0.01
- added link rotor_fl; visual sphere radius=0.03
- link base_link: geometry collision box size=0.2 0.2 0.05; visual box size=0.2 0.2 0.05
- link gps: geometry visual sphere radius=0.05
Joints:
- removed joint base_footprint_to_base_link
- removed joint base_link_to_gps_link
- added joint footprint_joint: type fixed, parent base_link, child base_footprint, origin xyz=0 0 0
- added joint gps_joint: type fixed, parent base_link, child gps, origin xyz=0 0 0.2
- added joint joint_bl: type fixed, parent base_link, child arm_bl, origin xyz=0 0 0
- added joint joint_br: type fixed, parent base_link, child arm_br, origin xyz=0 0 0
- added joint joint_fl: type fixed, parent base_link, child arm_fl, origin xyz=0 0 0
- added joint joint_fr: type fixed, parent base_link, child arm_fr, origin xyz=0 0 0
- added joint rotor_joint_fl: type fixed, parent arm_fl, child rotor_fl, origin xyz=0.15 0 0

Commit message: New Background

File: src/drone/urdf/robot.urdf (robot description, URDF)
Before this commit: robot simple_drone, 8 links, 7 joints
Links:
- added link cam_down_link; visual box size=0.05 0.05 0.02
Joints:
- added joint cam_down_joint: type fixed, parent base_link, child cam_down_link, origin xyz=0 0 -0.1 rpy=3.14159 0 -1.570795
